Commit message: Movimiento del robot

File: src/custom_pallet_gripper/urdf/pallet_gripper.urdf.xacro (robot description, xacro)
@@ -18,5 +18,5 @@
       <collision>
         <geometry>
-          <box size="0.1 0.1 0.1"/>
+          <box size="0.3 0.3 0.1"/>
         </geometry>
       </collision>
